File: hardware/sband_transmitter.kicad_pcb (KiCad board)
At the start: 8 copper layers, 91.7 x 88.7 mm, 430 parts, among them IC1 LMS7002M, IC10 LM75, IC11 DAC6311IDCK, IC12 M24128, IC13 LD39100PUR, IC14 LMZ20501SILR, IC15 W25Q128JVSIQ, IC16 AD5662, IC17 AS431, IC18 LD39100PUR, IC2 M24128, IC20 74LVC1G3157FZ4, IC3 SKY13411-374LF, IC4 SKY13411-374LF, IC5 LD39100PUR, IC6 LD39100PUR, IC7 LFE5U-45F-MG285, IC9 LMK00105, J10 PC104-Mainboard, J11 Conn_Coaxial, J13 Conn_Coaxial, J3 FPGA GPIO, J4 FPGA EGPIO (board edge), J5 FPGA JTAG (board edge), J7 U.FL/MMCX, J8 U.FL/MMCX, J9 FAN, T1 TC1-1-13M-45+, T2 TC1-1-13M-45+, T3 TC1-1-13M-45+, T4 TC1-1-13M-45+, U2 GRF5115, U3 GRF5115

Commit message: Linking schematics components to PCB
Parts:
- U3: footprint spacelab2:QFN-16_GRF -> library:QFN-16_GRF
